Commit message: openarm: correct v2 gripper finger joint travel to the motor's full range
The v2 URDF gave each pinch-gripper finger 0..0.7854 rad (45deg) of travel,
but the DM4310 motor commands 0..pi/2 and the fingers reach pi/2 at full open
(1:1 motor-to-finger, confirmed on hardware). The collision model and both sims
place the finger hulls straight from these URDF limits, so at 45deg they under-
splayed the open fingers and read clearance where the real fingers collided.

Set all four finger joints to +/-pi/2 and correct the openarm_can note that
described the ratio as unresolved.

File: openarm_description/assets/openarm_v20.urdf (robot description, URDF)
Before this commit: robot openarm_v20, 22 links, 21 joints
Joints:
- joint openarm_left_finger_joint1: limit lower=0 upper=0.7854 effort=7 velocity=5 -> lower=0 upper=1.5708 effort=7 velocity=5
- joint openarm_left_finger_joint2: limit lower=0 upper=0.7854 effort=7 velocity=5 -> lower=0 upper=1.5708 effort=7 velocity=5
- joint openarm_right_finger_joint1: limit lower=-0.7854 upper=0 effort=7 velocity=5 -> lower=-1.5708 upper=0 effort=7 velocity=5
- joint openarm_right_finger_joint2: limit lower=-0.7854 upper=0 effort=7 velocity=5 -> lower=-1.5708 upper=0 effort=7 velocity=5
