Commit message: openarm_description: the v2 pedestal carries its head camera
The OpenArm v2 mounts a ZED Mini on a bracket under a head cover, 63 mm
above the top of the torso mesh and in front of it, right where an arm
reaching overhead passes. The description carries the pedestal alone, so
the self-collision governor checks the arms against a torso whose
geometry stops below the camera, and the MuJoCo and Isaac robots draw a
camera from Waldo's pack that the governor governing them knows nothing
of.

The v2 URDF now mounts an `openarm_head_camera` link on the pedestal,
its collision geometry the convex hull of the ZED Mini, the bracket and
the cover, taken byte-identical from that same pinned pack with the
mount origin its rig gives. The hull straddles the top of the torso
mesh, so it rides its own link: the collision model fits a world-fixed
link as its own body, two world-fixed bodies never pair, and the arms
are checked against the camera and the torso separately.

The tests pin the placement: the hull's extents in the pedestal frame to
half a millimetre on every axis, and the two ZED lens fronts the pack
derives from the CAD inside it, so the geometry the governor keeps the
arms off is the geometry the camera looks out of. A v1 pedestal carries
no head camera.

Co-Authored-By: Claude Opus 5 (1M context) <noreply@anthropic.com>

File: openarm_description/assets/openarm_v20.urdf (robot description, URDF)
Before this commit: robot openarm_v20, 24 links, 23 joints
Links:
- added link openarm_head_camera; collision mesh filename=package://openarm_description/assets/meshes_v20/head_camera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 scale=1 1 1
Joints:
- added joint openarm_head_camera_mount_joint: type fixed, parent openarm_body_link0, child openarm_head_camera, origin xyz=0.0315 0 0.743 rpy=0 0 0
