Commit message: Control the gripper's grasp point, not the wrist it mounts on
An arm's end-effector was always its chain tip, so every caller with a gripper
carried the tip-to-grasp-point offset itself: onto a target before solving, off
a reported pose, and never at all on the Jacobian the speed limits and the
resolved-rate servo run on. Asking for an object's centre asked the arm to put
its wrist there and drive the gripper 16 cm through the table.

The URDFs gain the frame, because it is geometry: a fixed `openarm_{side}_tcp`
link off each chain tip, holding the grasp point with `+z` out of the gripper
along its approach direction and `y` on the jaw closing axis. Both are on the
gripping face, located by the jaw's own kinematics:

- v1's jaws are prismatic, the pads stay parallel at every opening, and an
  object meets the whole face, so the point is the face centre.
- v2's jaws are revolute, so opening splays the pads and the face tapers. An
  object wedges where the gap is narrowest, measured to be the pad's proximal
  edge for every object from 10 mm to the jaw's 65 mm limit, so the point is
  that pinch line rather than the face centre 5 mm ahead of it.

The generations mount their grippers along opposite tip axes, so v2's frame
carries a half turn about y and a caller writing a top-down grasp need not know
which generation it drives. v1's vendored `hand_tcp` link is renamed to `hand`:
it is the gravity feedforward's 0.127 kg hand-mass carrier sitting at identity
to link7, and a name that claims to be a TCP while resolving to the flange is
exactly the trap this change removes. The tests bracket the frame against the
bundled meshes, not against a second copy of itself: the point must sit midway
between the knuckles, on the gripping face (false in the relief behind the pad,
at the knuckle, and past the tip), with `+z` out of the gripper and `y` on the
closing axis.

srs_model mounts it by name. `with_tool_link` resolves a link that must sit
below the tip on fixed joints only, and the arm then speaks that frame
throughout: `ee_pose` reports it, the Jacobian is taken at it, `solve_ik` takes
targets in it, `rate_step` realizes twists at it. A link reached through a
movable joint is rejected, since its offset would silently track that joint.
The closed-form IK still needs the tip origin at the wrist center, so the SRS
model keeps deriving from the tip (`home_tip`, `Posed::tip_pose`) and
`solve_ik` strips the tool off the target before the solver sees it. Mounting
nothing leaves every existing consumer on the tip, so a dynamics-only caller
(an arm driver's gravity feedforward) is untouched.

openarm_description resolves the name per generation (`tcp_link`, beside
`base_link`), keeping it pure data.

Two things found while building it, fixed here because the tool frame reaches
both:

- A lower joint limit floor never reached the solver. `ArmModel` copied the
  limits when it was built, which is before any floor is layered on, so
  `limits()` reported the elbow's 0.05 floor while `solve_ik` kept returning
  configurations inside 2.9 degrees of straight, the singularity band the floor
  exists to avoid. Fixed by deleting the copy rather than syncing it: limits
  are the FK chain's and `ik::solve` now takes them live. Tool-frame targets
  sit closer to full extension, so this was about to get easier to hit.
- Manipulability is invariant under a rigid tool offset (the adjoint is
  unimodular), which is why the solver scores `MaxManipulability` on the
  tip-based PoE Jacobian while the servo runs on the tool-based one. Pinned by
  test, because the asymmetry otherwise reads as a bug worth "fixing".

File: openarm_description/assets/openarm_v10.urdf (robot description, URDF)
Before this commit: robot openarm, 24 links, 23 joints
Links:
- removed link openarm_left_hand_tcp
- removed link openarm_right_hand_tcp
- added link openarm_left_hand, mass 0.127
- added link openarm_left_tcp
- added link openarm_right_hand, mass 0.127
- added link openarm_right_tcp
Joints:
- removed joint openarm_left_hand_tcp_joint
- removed joint openarm_right_hand_tcp_joint
- added joint openarm_left_hand_joint: type fixed, parent openarm_left_link7, child openarm_left_hand, origin xyz=0 0 0 rpy=0 0 0
- added joint openarm_left_tcp_joint: type fixed, parent openarm_left_link7, child openarm_left_tcp, origin xyz=-0.0015 0 0.1717 rpy=0 0 0
- added joint openarm_right_hand_joint: type fixed, parent openarm_right_link7, child openarm_right_hand, origin xyz=0 0 0 rpy=0 0 0
- added joint openarm_right_tcp_joint: type fixed, parent openarm_right_link7, child openarm_right_tcp, origin xyz=-0.0015 0 0.1717 rpy=0 0 0

File: openarm_description/assets/openarm_v20.urdf (robot description, URDF)
Before this commit: robot openarm_v20, 22 links, 21 joints
Links:
- added link openarm_left_tcp
- added link openarm_right_tcp
Joints:
- added joint openarm_left_tcp_joint: type fixed, parent openarm_left_ee_base_link, child openarm_left_tcp, origin xyz=-0.0014 0 -0.16 rpy=0 3.141592653589793 0
- added joint openarm_right_tcp_joint: type fixed, parent openarm_right_ee_base_link, child openarm_right_tcp, origin xyz=-0.0014 0 -0.16 rpy=0 3.141592653589793 0

File: srs_model/tests/fixtures/openarm_v10.urdf (robot description, URDF)
Before this commit: robot openarm, 24 links, 23 joints
Links:
- removed link openarm_left_hand_tcp
- removed link openarm_right_hand_tcp
- added link openarm_left_hand
- added link openarm_left_tcp
- added link openarm_right_hand
- added link openarm_right_tcp
Joints:
- removed joint openarm_left_hand_tcp_joint
- removed joint openarm_right_hand_tcp_joint
- added joint openarm_left_hand_joint: type fixed, parent openarm_left_link7, child openarm_left_hand, origin xyz=0 0 0 rpy=0 0 0
- added joint openarm_left_tcp_joint: type fixed, parent openarm_left_link7, child openarm_left_tcp, origin xyz=-0.0015 0 0.1717 rpy=0 0 0
- added joint openarm_right_hand_joint: type fixed, parent openarm_right_link7, child openarm_right_hand, origin xyz=0 0 0 rpy=0 0 0
- added joint openarm_right_tcp_joint: type fixed, parent openarm_right_link7, child openarm_right_tcp, origin xyz=-0.0015 0 0.1717 rpy=0 0 0
